File: mainboard/Revision History.kicad_sch (KiCad schematic)
At the start: 0 parts

Commit message: Layout complete
Other:
- title: Template -> Revision History
Changed lines of the file:
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@@
 	(paper "A4")
 	(title_block
-		(title "Template")
+		(title "Revision History")
 		(date "2025-12-19")
 		(rev "1")
@@
 		)
 	)
-	(text_box "[${#}] ${TITLE}"
-		(exclude_from_sim no)
-		(at 80.01 16.51 0)
-		(size 137.16 12.7)
-		(margins 4.4999 4.4999 4.4999 4.4999)
-		(stroke
-			(width -0.0001)
-			(type default)
-		)
-		(fill
-			(type none)
-		)
-		(effects
-			(font
-				(face "Times New Roman")
-				(size 6 6)
-				(thickness 1.2)
-				(bold yes)
-				(color 162 22 34 1)
-			)
-		)
-	)
 	(text_box "${RELEASE_BODY_1.0.0}"
 		(exclude_from_sim no)
@@
 		)
 	)
+	(text_box "[${#}] ${TITLE}"
+		(exclude_from_sim no)
+		(at 12.7 12.7 0)
+		(size 271.78 20.32)
+		(margins 5.9999 5.9999 5.9999 5.9999)
+		(stroke
+			(width -0.0001)
+			(type default)
+		)
+		(fill
+			(type none)
+		)
+		(effects
+			(font
+				(face "Times New Roman")
+				(size 8 8)
+				(thickness 1.2)
+				(bold yes)
+				(color 162 22 34 1)
+			)
+		)
+	)
